Commit message: Modified URDF with real robot param and to consider collision with gripper and fingers

File: baxter_description/urdf/baxter_original.urdf (robot description, URDF)
Before this commit: robot baxter, 49 links, 48 joints
Links:
- link left_gripper_base: geometry visual box size=0.025 0.075 0.035
- link pedestal: geometry collision mesh filename=package://baxter_description/meshes/base/pedestal_link_coll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; visual mesh filename=package://baxter_description/meshes/base/PEDESTAL.DAE
- link right_gripper_base: geometry visual box size=0.025 0.075 0.035
- link torso: geometry collision mesh filename=package://baxter_description/meshes/torso/base_link_collisi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; visual mesh filename=package://baxter_description/meshes/torso/base_link.DAE
Joints:
- joint left_torso_arm_mount: origin xyz=0.0249978 0.218941 0.108059 rpy=-0.00240339 -0.00217116 0.783781 -> xyz=0.024645 0.219645 0.118588 rpy=0 0 0.7854
- joint right_torso_arm_mount: origin xyz=0.0246292 -0.219914 0.109009 rpy=-0.00170042 -0.00427862 -0.777907 -> xyz=0.024645 -0.219645 0.118588 rpy=0 0 -0.7854
