Commit message: URDF modified

File: baxter_description/urdf/baxter.urdf (robot description, URDF)
Before this commit: robot baxter, 49 links, 48 joints
Joints:
- joint collision_head_1: parent base -> torso
- joint collision_head_2: parent base -> torso
- joint torso_t0: origin xyz=0 0 0 rpy=0 0 0 -> xyz=0 0 0.93 rpy=0 0 0

Commit message: Added gripper with finger and its collision model in urdf

File: baxter_description/urdf/baxter.urdf (robot description, URDF)
Before this commit: robot baxter, 49 links, 48 joints
Links:
- added link camera_link, mass 0.0001
- link right_gripper_base: geometry collision cylinder length=0.062 radius=0.007; collision cylinder length=0.062 radius=0.007
Joints:
- added joint camera_link: type fixed, parent torso, child camera_link, origin xyz=0.0947 0 .6 rpy=0 0 0

Commit message: Modified baxter URDF

File: baxter_description/urdf/baxter.urdf (robot description, URDF)
Before this commit: robot baxter, 50 links, 49 joints
Links:
- removed link camera_link
Joints:
- removed joint camera_link
- joint right_endpoint: origin xyz=0.0 0 0.025 rpy=0 0 0 -> xyz=0.0 0 0.01 rpy=0 0 0

Commit message: Modifs on baxter's eef

File: baxter_description/urdf/baxter.urdf (robot description, URDF)
Before this commit: robot baxter, 50 links, 49 joints
Links:
- link right_gripper_base: geometry collision cylinder length=0.062 radius=0.01; collision cylinder length=0.062 radius=0.01
